File: KnxBoard.kicad_pcb (KiCad board)
At the start: 2 copper layers, 43.2 x 84.5 mm, 3 parts, among them P1 CONN28, P2 CONN28, P3 CONN6

Commit message: Update
Parts:
- removed P1, P2: CONN28, Connector_PinHeader_2.54mm:PinHeader_1x28_P2.54mm_Vertical
- removed P3: CONN6, Connector_PinHeader_2.54mm:PinHeader_1x06_P2.54mm_Vertical
- added C1: 100nF, Capacitor_SMD:C_0603_1608Metric, B.Cu at (101.6, 106.7)
- added C10: 100nF, Capacitor_SMD:C_0603_1608Metric, B.Cu at (128.8, 126.3)
- added C11: 47uF, Capacitor_SMD:C_0805_2012Metric, B.Cu at (107.1, 118.8)
- added C12: 100nF, Capacitor_SMD:C_0603_1608Metric, B.Cu at (124.8, 121.3)
- added C13: 100nF, Capacitor_SMD:C_0603_1608Metric, B.Cu at (132.1, 128.8)
- added C14: 1nF, Capacitor_SMD:C_0603_1608Metric, B.Cu at (120.0, 118.0)
- added C15: 100pF, Capacitor_SMD:C_0603_1608Metric, B.Cu at (124.8, 123.8)
- added C16: 22uF, Capacitor_SMD:C_0805_2012Metric, B.Cu at (123.9, 126.6)
- added C17: 47uF, Capacitor_SMD:C_0805_2012Metric, B.Cu at (111.5, 117.8)
- added C18: 22uF, Capacitor_SMD:C_0805_2012Metric, B.Cu at (127.9, 131.5)
- added C2: 100nF, Capacitor_SMD:C_0603_1608Metric, B.Cu at (83.8, 78.7)
- added C3: 47uF, Capacitor_SMD:C_0805_2012Metric, B.Cu at (119.1, 134.9)
- added C4: 100nF, Capacitor_SMD:C_0603_1608Metric, B.Cu at (118.9, 132.2)
- added C5: 470nF, Capacitor_SMD:C_0603_1608Metric, B.Cu at (128.1, 128.8)
- added C6: 10nF, Capacitor_SMD:C_0603_1608Metric, B.Cu at (120.5, 120.9)
- added C7: 100uF, Capacitor_SMD:CP_Elec_6.3x7.7, F.Cu at (83.8, 94.0)
- added C8: 47nF, Capacitor_SMD:C_0603_1608Metric, B.Cu at (128.8, 123.8)
- added C9: 47nF, Capacitor_SMD:C_0603_1608Metric, B.Cu at (124.0, 118.4)
- added D1: SMAJ40CA, Diode_SMD:D_SMA, F.Cu at (91.4, 109.2)
- added D2: 1N4148, Diode_SMD:D_SOD-323, B.Cu at (120.6, 123.6)
- added D3: 1N4148, Diode_SMD:D_SOD-323, B.Cu at (115.9, 117.8)
- added D4: 1N4148, Diode_SMD:D_SOD-323, B.Cu at (132.2, 131.5)
- added J1: SB, Connector_PinHeader_2.54mm:PinHeader_1x02_P2.54mm_Vertical, F.Cu at (94.0, 94.0)
- added J2: KNX, stknx:KNX_Connector, F.Cu at (91.4, 116.8)
- added J3: Conn_01x14, Connector_PinHeader_2.54mm:PinHeader_1x14_P2.54mm_Vertical, F.Cu at (109.2, 111.8)
- added J4: Conn_01x02, Connector_PinHeader_2.54mm:PinHeader_1x02_P2.54mm_Vertical, F.Cu at (83.8, 111.8)
- added J5: Conn_01x14, Connector_PinHeader_2.54mm:PinHeader_1x14_P2.54mm_Vertical, F.Cu at (76.2, 78.7)
- added L1: 33uH, Inductor_SMD:L_Taiyo-Yuden_NR-40xx, F.Cu at (101.6, 88.9)
- added L2: 33uH, Inductor_SMD:L_Taiyo-Yuden_NR-40xx, F.Cu at (81.3, 101.6)
- added LD1: LED, LED_SMD:LED_0603_1608Metric, F.Cu at (99.1, 104.1)
- added R1: 100R, Resistor_SMD:R_0402_1005Metric, F.Cu at (99.1, 101.6)
- added R2: 10K, Resistor_SMD:R_0402_1005Metric, B.Cu at (101.5, 124.6)
- added R3: 4.7M, Resistor_SMD:R_0402_1005Metric, B.Cu at (127.5, 119.1)
- added R4: 68R, Resistor_SMD:R_0612_1632Metric, F.Cu at (94.0, 101.6)
- added R5: 1K, Resistor_SMD:R_0402_1005Metric, B.Cu at (128.2, 121.5)
- added R6: 1K, Resistor_SMD:R_0402_1005Metric, B.Cu at (132.2, 124.5)
- added R7: 10K, Resistor_SMD:R_0402_1005Metric, B.Cu at (131.1, 121.5)
- added R8: 110K, Resistor_SMD:R_0402_1005Metric, B.Cu at (132.2, 126.5)
- added SW1: SW, Button_Switch_SMD:SW_SPST_SKQG_WithStem, F.Cu at (101.6, 109.2)
- added SW2: SW, Button_Switch_SMD:SW_SPST_SKQG_WithStem, F.Cu at (83.8, 81.3)
- added U1: STM32L432KCUx, Package_DFN_QFN:QFN-32-1EP_5x5mm_P0.5mm_EP3.45x3.45mm, F.Cu at (94.0, 83.8)
- added U2: STKNX, Package_DFN_QFN:VQFN-24-1EP_4x4mm_P0.5mm_EP2.45x2.45mm_ThermalVias, F.Cu at (88.9, 101.6)
- added X1: SG-3030CM, Oscillator:Oscillator_SMD_SeikoEpson_SG3030CM, F.Cu at (104.1, 78.7)
Routing:
- removed copper zone on B.Cu, net GND
Other:
- board outline removed
- net class Default: clearance 0.254 -> 0.2; trace_width 0.254 -> 0.25; via_dia 0.889 -> 0.8; via_drill 0.635 -> 0.4
- rule trace_clearance: 0.254 -> 0.2
- rule trace_min: 0.254 -> 0.2
- rule via_min_drill: 0.508 -> 0.3
- rule via_min_size: 0.889 -> 0.4
- board text removed: "STM32 Value Line Discovery - Shield"
