File: KnxBoard.kicad_pcb (KiCad board)
At the start: 4 copper layers, 35.8 x 33.8 mm, 44 parts, among them IC1 STM32G491KEU6, IC2 NCN5130MNTWG, J1 Conn_01x02, J2 Conn_02x03_Counter_Clockwise, J3 Conn_01x10, J4 Conn_01x10, SW1 SW_Push, Y1 16MHz

Commit message: Add NRST and 3V3 to debug connector
Connect ANAOUT to STM ADC to be able to support the KNX System B standard

Update to kicad 10.0
Connections:
- IC2 pad 39: unconnected-(IC2-ANAOUT-Pad39) -> Net-(IC1-PB0)
- J2 pad 3: GND -> Net-(IC1-PG10-NRST)
- J2 pad 6: Net-(IC1-DEBUG_RX) -> 3V3
- J4 pad 3: Net-(IC1-PB0) -> unconnected-(J4-Pin_3-Pad3)
Routing:
- net Net-(IC1-PB0): track 12.3 -> 27.0 mm, vias 0 -> 2
- net Net-(IC1-PG10-NRST): track 35.7 -> 41.5 mm
- net 3V3: track 79.3 -> 83.4 mm, vias 8 -> 9
- net Net-(IC1-DEBUG_RX): track 26.0 -> 22.6 mm, vias 0 -> 1
- net Net-(IC1-PA12): track 21.3 -> 23.1 mm
- net GND: track 68.7 -> 67.5 mm
Other:
- board text added: "PB0"
