File: stknx.sch (KiCad schematic (older format))
At the start: 26 parts, among them U1 STKNX

Commit message: Work on componant sources
Parts:
- C1: value 100nF 6.3V -> 100nF; Price (none) -> 0.09; Rating (none) -> 6.3V; STKNX (none) -> CSS
- C10: value 10nF 50V -> 10nF; footprint Resistor_SMD:R_0603_1608Metric -> Capacitor_SMD:C_0603_1608Metric; Price (none) -> 0.09; Rating (none) -> 50V; STKNX (none) -> CAC
- C11: value 100nF 50V -> 100nF; footprint Resistor_SMD:R_0603_1608Metric -> Capacitor_SMD:C_0603_1608Metric; Price (none) -> 0.09; Rating (none) -> 50V; STKNX (none) -> CPH
- C12: value 1nF 5V -> 1nF; Price (none) -> 0.23; Rating (none) -> 5V
- C13: value 100nF 50V -> 100nF; footprint Resistor_SMD:R_0603_1608Metric -> Capacitor_SMD:C_0603_1608Metric; Price (none) -> 0.09; Rating (none) -> 50V; STKNX (none) -> CPL
- C2: value 100pF 16V -> 100pF; Price (none) -> 0.04; Rating (none) -> 16V; STKNX (none) -> CFB1
- C21: value 4.7uF 6.3V -> 47uF; footprint Resistor_SMD:R_0603_1608Metric -> Capacitor_SMD:C_0805_2012Metric; Price (none) -> 0.82; Rating (none) -> 3.3V; STKNX (none) -> CCORE
- C3: value 47uF 10V -> 47uF; footprint Capacitor_SMD:C_0603_1608Metric -> Capacitor_SMD:C_0805_2012Metric; Price (none) -> 0.82; Rating (none) -> 10V; STKNX (none) -> CGATE
- C4: value 470nF 35V -> 470nF; footprint Resistor_SMD:R_0603_1608Metric -> Capacitor_SMD:C_0603_1608Metric; Price (none) -> 0.21; Rating (none) -> 35V; STKNX (none) -> CREF
- C5: value 10uF 35V -> 22uF; footprint Capacitor_SMD:C_0603_1608Metric -> Capacitor_SMD:C_0805_2012Metric; Price (none) -> 1.03; Rating (none) -> 35V; STKNX (none) -> CIN
- C6: value 22uF 25V -> 22uF; footprint Resistor_SMD:R_0603_1608Metric -> Capacitor_SMD:C_0805_2012Metric; Price (none) -> 1.03; Rating (none) -> 12V; STKNX (none) -> COUT
- C7: value 100uF 35V -> 100uF; Rating (none) -> 35V; STKNX (none) -> CVDDHV
- C8: value 47nF 35V -> 47nF; footprint Resistor_SMD:R_0603_1608Metric -> Capacitor_SMD:C_0603_1608Metric; Price (none) -> 0.24; Rating (none) -> 35V; STKNX (none) -> CFH
- C9: value 47nF 35V -> 47nF; footprint Resistor_SMD:R_0603_1608Metric -> Capacitor_SMD:C_0603_1608Metric; Price (none) -> 0.24; Rating (none) -> 35V; STKNX (none) -> CFL
- D1, D3, D4: Price (none) -> 0.13
- D2: Price (none) -> 0.32
- L1: value L -> 33uH; footprint Inductor_SMD:L_1210_3225Metric -> Inductor_SMD:L_Taiyo-Yuden_NR-40xx; Price (none) -> 0.41; Rating (none) -> Ir > 150mA Isat > 550mA; STKNX (none) -> L
Connections:
- wire segments 103 -> 104
Other:
- moved on the sheet: C13

Commit message: Work on BOM
Parts:
- C7: footprint Capacitor_SMD:C_Elec_6.3x7.7 -> Capacitor_SMD:CP_Elec_6.3x7.7; Price (none) -> 0.43
- R3: renamed from R5; Price (none) -> 0.09
- R4: renamed from R3; footprint Resistor_SMD:R_1218_3246Metric -> Resistor_SMD:R_0612_1632Metric; Price (none) -> 0.43; Rating (none) -> 1W; STKNX (none) -> RTX
- R5: renamed from R4; Price (none) -> 0.09
- R6: Price (none) -> 0.09
- R7: renamed from R2; Price (none) -> 0.09
- R8: renamed from R1; Price (none) -> 0.09
- U2: renamed from U1; Price (none) -> 3.82
- renumbered C11 to C10, C3 to C11, C13 to C12, C1 to C13, C12 to C14, C2 to C15, C5 to C16, C21 to C17, C6 to C18, C4 to C5, C10 to C6, C9 to C8, C8 to C9, D2 to D1, D1 to D2, L1 to L2
Changed lines of the file:
@@
 $EndDescr
 $Comp
-L ${KIPRJMOD}/local/stknx.lib:STKNX U1
+L ${KIPRJMOD}/local/stknx.lib:STKNX U2
 U 1 1 5ECBF041
 P 5250 3500
-F 0 "U1" H 5150 4050 50  0000 C CNN
+F 0 "U2" H 5150 4050 50  0000 C CNN
 F 1 "STKNX" H 5150 3900 50  0000 C CNN
 F 2 "Package_DFN_QFN:VQFN-24-1EP_4x4mm_P0.5mm_EP2.45x2.45mm_ThermalVias" H 3800 3000 50  0001 C CNN
-F 3 "" H 3800 3000 50  0001 C CNN
+F 3 "https://www.mouser.fr/ProductDetail/STMicroelectronics/STKNXTR?qs=lYGu3FyN48cC0CqtOx84%252BQ%3D%3D" H 3800 3000 50  0001 C CNN
+F 4 "3.82" H 5250 3500 50  0001 C CNN "Price"
 	1    5250 3500
 	1    0    0    -1
 $EndComp
 $Comp
-L Device:R R4
+L Device:R R5
 U 1 1 5ECC0BB4
 P 3450 4300
-F 0 "R4" V 3243 4300 50  0000 C CNN
+F 0 "R5" V 3243 4300 50  0000 C CNN
 F 1 "1K" V 3334 4300 50  0000 C CNN
 F 2 "Resistor_SMD:R_0603_1608Metric" V 3380 4300 50  0001 C CNN
-F 3 "~" H 3450 4300 50  0001 C CNN
+F 3 "https://www.mouser.fr/ProductDetail/Vishay-Dale/CRCW06031K00FKEAC?qs=sGAEpiMZZMvdGkrng054t0DrEhLhGh8g1B5lDmmPZz5NoSHbyVr1tg%3D%3D" H 3450 4300 50  0001 C CNN
+F 4 "0.09" H 3450 4300 50  0001 C CNN "Price"
 	1    3450 4300
 	0    1    1    0
@@
 F 1 "1K" H 3630 4845 50  0000 R CNN
 F 2 "Resistor_SMD:R_0603_1608Metric" V 3630 4800 50  0001 C CNN
-F 3 "~" H 3700 4800 50  0001 C CNN
+F 3 "https://www.mouser.fr/ProductDetail/Vishay-Dale/CRCW06031K00FKEAC?qs=sGAEpiMZZMvdGkrng054t0DrEhLhGh8g1B5lDmmPZz5NoSHbyVr1tg%3D%3D" H 3700 4800 50  0001 C CNN
+F 4 "0.09" H 3700 4800 50  0001 C CNN "Price"
 	1    3700 4800
 	-1   0    0    1
 $EndComp
 $Comp
-L Device:C C13
+L Device:C C12
 U 1 1 5ECC2867
 P 3700 5200
-F 0 "C13" H 3585 5154 50  0000 R CNN
+F 0 "C12" H 3585 5154 50  0000 R CNN
 F 1 "100nF" H 3585 5245 50  0000 R CNN
 F 2 "Capacitor_SMD:C_0603_1608Metric" H 3738 5050 50  0001 C CNN
@@
 $EndComp
 $Comp
-L Device:R R3
+L Device:R R4
 U 1 1 5ECC7B6F
 P 3450 3900
-F 0 "R3" V 3657 3900 50  0000 C CNN
+F 0 "R4" V 3657 3900 50  0000 C CNN
 F 1 "68R" V 3566 3900 50  0000 C CNN
-F 2 "Resistor_SMD:R_1218_3246Metric" V 3380 3900 50  0001 C CNN
-F 3 "~" H 3450 3900 50  0001 C CNN
+F 2 "Resistor_SMD:R_0612_1632Metric" V 3380 3900 50  0001 C CNN
+F 3 "https://www.mouser.fr/ProductDetail/Vishay-Beyschlag/MCW0612MC6809FP100?qs=sGAEpiMZZMvdGkrng054twGMB1RJ6An1VEdxKzVKfLNKDpMMSDfotA%3D%3D" H 3450 3900 50  0001 C CNN
+F 4 "1W" H 3450 3900 50  0001 C CNN "Rating"
+F 5 "RTX" H 3450 3900 50  0001 C CNN "STKNX"
+F 6 "0.43" H 3450 3900 50  0001 C CNN "Price"
 	1    3450 3900
 	0    -1   -1   0
 $EndComp
 $Comp
-L Device:C C3
+L Device:C C11
 U 1 1 5ECC838F
 P 3450 2300
-F 0 "C3" V 3702 2300 50  0000 C CNN
+F 0 "C11" V 3702 2300 50  0000 C CNN
 F 1 "47uF" V 3611 2300 50  0000 C CNN
 F 2 "Capacitor_SMD:C_0805_2012Metric" H 3488 2150 50  0001 C CNN
@@
 $EndComp
 $Comp
-L Device:D D1
+L Device:D D2
 U 1 1 5ECCCDFA
 P 1600 4100
-F 0 "D1" H 1600 4316 50  0000 C CNN
+F 0 "D2" H 1600 4316 50  0000 C CNN
 F 1 "1N4148" H 1600 4225 50  0000 C CNN
 F 2 "Diode_SMD:D_SOD-323" H 1600 4100 50  0001 C CNN
@@
 $EndComp
 $Comp
-L Device:D_TVS D2
+L Device:D_TVS D1
 U 1 1 5ECCF534
 P 1300 5050
-F 0 "D2" V 1254 5129 50  0000 L CNN
+F 0 "D1" V 1254 5129 50  0000 L CNN
 F 1 "SMAJ40CA" V 1345 5129 50  0000 L CNN
 F 2 "Diode_SMD:D_SMA" H 1300 5050 50  0001 C CNN
@@
 $EndComp
 $Comp
-L power:GNDREF #PWR0107
+L power:GNDREF #PWR06
 U 1 1 5ECD1541
 P 3700 5650
-F 0 "#PWR0107" H 3700 5400 50  0001 C CNN
+F 0 "#PWR06" H 3700 5400 50  0001 C CNN
 F 1 "GNDREF" H 3705 5477 50  0000 C CNN
 F 2 "" H 3700 5650 50  0001 C CNN
@@
 	3700 4550 3800 4550
 $Comp
-L Device:R R5
+L Device:R R3
 U 1 1 5ECD673E
 P 1900 5000
-F 0 "R5" H 1830 4954 50  0000 R CNN
+F 0 "R3" H 1830 4954 50  0000 R CNN
 F 1 "4.7M" H 1830 5045 50  0000 R CNN
 F 2 "Resistor_SMD:R_0603_1608Metric" V 1830 5000 50  0001 C CNN
-F 3 "~" H 1900 5000 50  0001 C CNN
+F 3 "https://www.mouser.fr/ProductDetail/Vishay-Dale/CRCW06034M70FKEA?qs=sGAEpiMZZMvdGkrng054tw79ugaueG8BzI1%2F17vrqTk%3D" H 1900 5000 50  0001 C CNN
+F 4 "0.09" H 1900 5000 50  0001 C CNN "Price"
 	1    1900 5000
 	-1   0    0    1
@@
 Connection ~ 1900 5400
 $Comp
-L Device:C C10
+L Device:C C6
 U 1 1 5ECE760D
 P 1750 3500
-F 0 "C10" V 2002 3500 50  0000 C CNN
+F 0 "C6" V 2002 3500 50  0000 C CNN
 F 1 "10nF" V 1911 3500 50  0000 C CNN
 F 2 "Capacitor_SMD:C_0603_1608Metric" H 1788 3350 50  0001 C CNN
@@
 	2500 5400 3700 5400
 $Comp
-L Device:C C8
+L Device:C C9
 U 1 1 5ECF37B0
 P 2800 2950
-F 0 "C8" V 2950 2950 50  0000 C CNN
+F 0 "C9" V 2950 2950 50  0000 C CNN
 F 1 "47nF" V 3050 3000 50  0000 C CNN
 F 2 "Capacitor_SMD:C_0603_1608Metric" H 2838 2800 50  0001 C CNN
@@
 F 0 "C7" V 2000 2800 50  0000 L CNN
 F 1 "100uF" V 2100 2550 50  0000 L CNN
-F 2 "Capacitor_SMD:C_Elec_6.3x7.7" H 2288 2700 50  0001 C CNN
-F 3 "~" H 2250 2850 50  0001 C CNN
+F 2 "Capacitor_SMD:CP_Elec_6.3x7.7" H 2288 2700 50  0001 C CNN
+F 3 "https://www.mouser.fr/ProductDetail/Nichicon/UUR1V101MCL6GS?qs=huzeVNXgovWypttWSImRTA%3D%3D" H 2250 2850 50  0001 C CNN
 F 4 "35V" H 2250 2850 50  0001 C CNN "Rating"
 F 5 "CVDDHV" V 2250 2850 50  0001 C CNN "STKNX"
+F 6 "0.43" H 2250 2850 50  0001 C CNN "Price"
 	1    2250 2850
 	1    0    0    -1
@@
 VDDHV
 $Comp
-L Device:C C4
+L Device:C C5
 U 1 1 5EDCEF61
 P 1400 2900
-F 0 "C4" V 1550 2900 50  0000 C CNN
+F 0 "C5" V 1550 2900 50  0000 C CNN
 F 1 "470nF" V 1650 2950 50  0000 C CNN
 F 2 "Capacitor_SMD:C_0603_1608Metric" H 1438 2750 50  0001 C CNN
@@
 KNX_TX
 $Comp
-L Device:C C12
+L Device:C C14
 U 1 1 5EDDD2EF
 P 6900 4500
-F 0 "C12" V 6750 4500 50  0000 C CNN
+F 0 "C14" V 6750 4500 50  0000 C CNN
 F 1 "1nF" V 6650 4450 50  0000 C CNN
 F 2 "Capacitor_SMD:C_0603_1608Metric" H 6938 4350 50  0001 C CNN
@@
 Connection ~ 7850 5400
 $Comp
-L Device:L L1
+L Device:L L2
 U 1 1 5EDEDD4C
 P 7200 2600
-F 0 "L1" V 7390 2600 50  0000 C CNN
+F 0 "L2" V 7390 2600 50  0000 C CNN
 F 1 "33uH" V 7299 2600 50  0000 C CNN
 F 2 "Inductor_SMD:L_Taiyo-Yuden_NR-40xx" H 7200 2600 50  0001 C CNN
@@
 	7550 3050 7550 3250
 $Comp
-L Device:C C6
+L Device:C C18
 U 1 1 5EDFDBE7
 P 8300 3700
-F 0 "C6" H 8150 3650 50  0000 R CNN
+F 0 "C18" H 8150 3650 50  0000 R CNN
 F 1 "22uF" H 8150 3750 50  0000 R CNN
 F 2 "Capacitor_SMD:C_0805_2012Metric" H 8338 3550 50  0001 C CNN
@@
 	8450 1250 8450 2900
 $Comp
-L Device:R R2
+L Device:R R7
 U 1 1 5EE165BA
 P 7550 1550
-F 0 "R2" V 7757 1550 50  0000 C CNN
+F 0 "R7" V 7757 1550 50  0000 C CNN
 F 1 "10K" V 7666 1550 50  0000 C CNN
 F 2 "Resistor_SMD:R_0603_1608Metric" V 7480 1550 50  0001 C CNN
-F 3 "~" H 7550 1550 50  0001 C CNN
+F 3 "https://www.mouser.fr/ProductDetail/Vishay-Dale/CRCW060310K0FKEA?qs=sGAEpiMZZMvdGkrng054t%252B8cnVAnHPZkqchqPaQRdrE%3D" H 7550 1550 50  0001 C CNN
+F 4 "0.09" H 7550 1550 50  0001 C CNN "Price"
 	1    7550 1550
 	1    0    0    -1
 $EndComp
 $Comp
-L Device:R R1
+L Device:R R8
 U 1 1 5EE16EF4
 P 7550 1950
-F 0 "R1" V 7757 1950 50  0000 C CNN
+F 0 "R8" V 7757 1950 50  0000 C CNN
 F 1 "110K" V 7666 1950 50  0000 C CNN
 F 2 "Resistor_SMD:R_0603_1608Metric" V 7480 1950 50  0001 C CNN
-F 3 "~" H 7550 1950 50  0001 C CNN
+F 3 "https://www.mouser.fr/ProductDetail/Vishay-Dale/CRCW0603110KFKEA?qs=sGAEpiMZZMvdGkrng054tz1PN3csf7M2czfciwwJb%252Bg%3D" H 7550 1950 50  0001 C CNN
+F 4 "0.09" H 7550 1950 50  0001 C CNN "Price"
 	1    7550 1950
 	1    0    0    -1
@@
 	7550 1750 7550 1800
 $Comp
-L Device:C C2
+L Device:C C15
 U 1 1 5EE22DE3
 P 7300 1950
-F 0 "C2" V 7150 1950 50  0000 C CNN
+F 0 "C15" V 7150 1950 50  0000 C CNN
 F 1 "100pF" V 7050 1900 50  0000 C CNN
 F 2 "Capacitor_SMD:C_0603_1608Metric" H 7338 1800 50  0001 C CNN
@@
 Connection ~ 8900 5400
 $Comp
-L Device:C C21
+L Device:C C17
 U 1 1 5EE4D481
 P 7850 3700
-F 0 "C21" H 8100 3650 50  0000 R CNN
+F 0 "C17" H 8100 3650 50  0000 R CNN
 F 1 "47uF" H 8150 3750 50  0000 R CNN
 F 2 "Capacitor_SMD:C_0805_2012Metric" H 7888 3550 50  0001 C CNN
@@
 $EndComp
 $Comp
-L Device:C C5
+L Device:C C16
 U 1 1 5EE51135
 P 7850 2650
-F 0 "C5" H 7700 2600 50  0000 R CNN
+F 0 "C16" H 7700 2600 50  0000 R CNN
 F 1 "22uF" H 7700 2700 50  0000 R CNN
 F 2 "Capacitor_SMD:C_0805_2012Metric" H 7888 2500 50  0001 C CNN
@@
 	3700 5350 3700 5400
 $Comp
-L Device:C C11
+L Device:C C10
 U 1 1 5EE5F286
 P 3050 4300
-F 0 "C11" H 2935 4254 50  0000 R CNN
+F 0 "C10" H 2935 4254 50  0000 R CNN
 F 1 "100nF" H 2935 4345 50  0000 R CNN
 F 2 "Capacitor_SMD:C_0603_1608Metric" H 3088 4150 50  0001 C CNN
@@
 $EndComp
 $Comp
-L Device:C C1
+L Device:C C13
 U 1 1 5EE64576
 P 5750 1700
-F 0 "C1" H 5635 1654 50  0000 R CNN
+F 0 "C13" H 5635 1654 50  0000 R CNN
 F 1 "100nF" H 5635 1745 50  0000 R CNN
 F 2 "Capacitor_SMD:C_0603_1608Metric" H 5788 1550 50  0001 C CNN
@@
 $EndComp
 $Comp
-L Device:C C9
+L Device:C C8
 U 1 1 5EE3FF32
 P 2650 3200
-F 0 "C9" V 2800 3200 50  0000 C CNN
+F 0 "C8" V 2800 3200 50  0000 C CNN
 F 1 "47nF" V 2900 3250 50  0000 C CNN
 F 2 "Capacitor_SMD:C_0603_1608Metric" H 2688 3050 50  0001 C CNN

Commit message: Resistors in 0402
Parts:
- R3, R5, R6, R7, R8: footprint Resistor_SMD:R_0603_1608Metric -> Resistor_SMD:R_0402_1005Metric
Changed lines of the file:
@@
 F 0 "R5" V 3243 4300 50  0000 C CNN
 F 1 "1K" V 3334 4300 50  0000 C CNN
-F 2 "Resistor_SMD:R_0603_1608Metric" V 3380 4300 50  0001 C CNN
-F 3 "https://www.mouser.fr/ProductDetail/Vishay-Dale/CRCW06031K00FKEAC?qs=sGAEpiMZZMvdGkrng054t0DrEhLhGh8g1B5lDmmPZz5NoSHbyVr1tg%3D%3D" H 3450 4300 50  0001 C CNN
+F 2 "Resistor_SMD:R_0402_1005Metric" V 3380 4300 50  0001 C CNN
+F 3 "https://www.mouser.fr/ProductDetail/Vishay-Dale/CRCW04021K00FKEDC?qs=sGAEpiMZZMvdGkrng054t0DrEhLhGh8gZ6wm0HkRlDUT6OA9YCnj9w%3D%3D" H 3450 4300 50  0001 C CNN
 F 4 "0.09" H 3450 4300 50  0001 C CNN "Price"
 	1    3450 4300
@@
 F 0 "R6" H 3630 4754 50  0000 R CNN
 F 1 "1K" H 3630 4845 50  0000 R CNN
-F 2 "Resistor_SMD:R_0603_1608Metric" V 3630 4800 50  0001 C CNN
-F 3 "https://www.mouser.fr/ProductDetail/Vishay-Dale/CRCW06031K00FKEAC?qs=sGAEpiMZZMvdGkrng054t0DrEhLhGh8g1B5lDmmPZz5NoSHbyVr1tg%3D%3D" H 3700 4800 50  0001 C CNN
+F 2 "Resistor_SMD:R_0402_1005Metric" V 3630 4800 50  0001 C CNN
+F 3 "https://www.mouser.fr/ProductDetail/Vishay-Dale/CRCW04021K00FKEDC?qs=sGAEpiMZZMvdGkrng054t0DrEhLhGh8gZ6wm0HkRlDUT6OA9YCnj9w%3D%3D" H 3700 4800 50  0001 C CNN
 F 4 "0.09" H 3700 4800 50  0001 C CNN "Price"
 	1    3700 4800
@@
 F 0 "R3" H 1830 4954 50  0000 R CNN
 F 1 "4.7M" H 1830 5045 50  0000 R CNN
-F 2 "Resistor_SMD:R_0603_1608Metric" V 1830 5000 50  0001 C CNN
-F 3 "https://www.mouser.fr/ProductDetail/Vishay-Dale/CRCW06034M70FKEA?qs=sGAEpiMZZMvdGkrng054tw79ugaueG8BzI1%2F17vrqTk%3D" H 1900 5000 50  0001 C CNN
+F 2 "Resistor_SMD:R_0402_1005Metric" V 1830 5000 50  0001 C CNN
+F 3 "https://www.mouser.fr/ProductDetail/Vishay-Dale/CRCW04024M70FKED?qs=sGAEpiMZZMvdGkrng054tx3Kv%252BhbWMRFX7ZUO10KL6w%3D" H 1900 5000 50  0001 C CNN
 F 4 "0.09" H 1900 5000 50  0001 C CNN "Price"
 	1    1900 5000
@@
 F 0 "R7" V 7757 1550 50  0000 C CNN
 F 1 "10K" V 7666 1550 50  0000 C CNN
-F 2 "Resistor_SMD:R_0603_1608Metric" V 7480 1550 50  0001 C CNN
-F 3 "https://www.mouser.fr/ProductDetail/Vishay-Dale/CRCW060310K0FKEA?qs=sGAEpiMZZMvdGkrng054t%252B8cnVAnHPZkqchqPaQRdrE%3D" H 7550 1550 50  0001 C CNN
+F 2 "Resistor_SMD:R_0402_1005Metric" V 7480 1550 50  0001 C CNN
+F 3 "https://www.mouser.fr/ProductDetail/Vishay-Dale/CRCW040210K0FKEDC?qs=sGAEpiMZZMvdGkrng054t0DrEhLhGh8ghRTPC4LoFoV0V5heIyAs3Q%3D%3D" H 7550 1550 50  0001 C CNN
 F 4 "0.09" H 7550 1550 50  0001 C CNN "Price"
 	1    7550 1550
@@
 F 0 "R8" V 7757 1950 50  0000 C CNN
 F 1 "110K" V 7666 1950 50  0000 C CNN
-F 2 "Resistor_SMD:R_0603_1608Metric" V 7480 1950 50  0001 C CNN
-F 3 "https://www.mouser.fr/ProductDetail/Vishay-Dale/CRCW0603110KFKEA?qs=sGAEpiMZZMvdGkrng054tz1PN3csf7M2czfciwwJb%252Bg%3D" H 7550 1950 50  0001 C CNN
+F 2 "Resistor_SMD:R_0402_1005Metric" V 7480 1950 50  0001 C CNN
+F 3 "https://www.mouser.fr/ProductDetail/Vishay-Dale/CRCW0402110KFKED?qs=sGAEpiMZZMvdGkrng054txEw7b1YnvGuJRsoX62K%252BYM%3D" H 7550 1950 50  0001 C CNN
 F 4 "0.09" H 7550 1950 50  0001 C CNN "Price"
 	1    7550 1950
