File: KnxBoard.kicad_sch (KiCad schematic)
At the start: 41 parts, among them IC1 STM32G491KEU6, IC2 NCN5130MNTWG, J1 Conn_01x02, J2 Conn_02x03_Counter_Clockwise, J3 Conn_01x10, J4 Conn_01x10, SW1 SW_Push, Y1 16MHz

Commit message: Route
Parts:
- IC1: footprint Library:QFN50P500X500X60-33N-D -> Package_DFN_QFN:UQFN-32_5x5mm_P0.5mm
- J2: footprint Connector_PinHeader_2.54mm:PinHeader_2x03_P2.54mm_Vertical -> Connector_PinHeader_1.27mm:PinHeader_2x03_P1.27mm_Vertical
- Y1: footprint Crystal:Crystal_SMD_3225-4Pin_3.2x2.5mm_HandSoldering -> Crystal:Crystal_SMD_3225-4Pin_3.2x2.5mm
Connections:
- net at J2.2 (Pin_2): now also IC1.23 (SYS_JTMS-SWDIO); no longer IC1.26 (DEBUG_TX)
- net at J2.3 (Pin_3): no longer IC1.25 (DEBUG_RX)
- net at J2.5 (Pin_5): now also IC1.26 (DEBUG_TX); no longer IC1.23 (SYS_JTMS-SWDIO)
- net at J2.6 (Pin_6): now also IC1.25 (DEBUG_RX)
Other:
- moved on the sheet: J2
Changed lines of the file:
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@@
 	)
 	(junction
-		(at 180.34 54.61)
-		(diameter 0)
-		(color 0 0 0 0)
-	)
-	(junction
 		(at 212.09 125.73)
 		(diameter 0)
@@
 	)
 	(junction
+		(at 215.9 54.61)
+		(diameter 0)
+		(color 0 0 0 0)
+	)
+	(junction
 		(at 226.06 115.57)
 		(diameter 0)
@@
 	)
 	(no_connect
-		(at 217.17 41.91)
+		(at 215.9 41.91)
 	)
 	(wire
@@
 	(wire
 		(pts
-			(xy 200.66 46.99) (xy 200.66 66.04)
-		)
-		(stroke
-			(width 0)
-			(type default)
-		)
-	)
-	(wire
-		(pts
 			(xy 60.96 49.53) (xy 49.53 49.53)
 		)
@@
 	(wire
 		(pts
+			(xy 215.9 54.61) (xy 246.38 54.61)
+		)
+		(stroke
+			(width 0)
+			(type default)
+		)
+	)
+	(wire
+		(pts
 			(xy 151.13 85.09) (xy 151.13 106.68)
 		)
@@
 	(wire
 		(pts
+			(xy 220.98 39.37) (xy 203.2 39.37)
+		)
+		(stroke
+			(width 0)
+			(type default)
+		)
+	)
+	(wire
+		(pts
 			(xy 88.9 135.89) (xy 91.44 135.89)
 		)
@@
 	(wire
 		(pts
+			(xy 215.9 46.99) (xy 215.9 54.61)
+		)
+		(stroke
+			(width 0)
+			(type default)
+		)
+	)
+	(wire
+		(pts
 			(xy 68.58 118.11) (xy 68.58 135.89)
 		)
@@
 	(wire
 		(pts
-			(xy 217.17 44.45) (xy 222.25 44.45)
-		)
-		(stroke
-			(width 0)
-			(type default)
-		)
-	)
-	(wire
-		(pts
 			(xy 104.14 133.35) (xy 104.14 143.51)
 		)
@@
 	(wire
 		(pts
-			(xy 180.34 54.61) (xy 246.38 54.61)
+			(xy 180.34 54.61) (xy 215.9 54.61)
 		)
 		(stroke
@@
 	(wire
 		(pts
-			(xy 204.47 41.91) (xy 180.34 41.91)
-		)
-		(stroke
-			(width 0)
-			(type default)
-		)
-	)
-	(wire
-		(pts
 			(xy 69.85 29.21) (xy 69.85 44.45)
 		)
@@
 	(wire
 		(pts
-			(xy 222.25 44.45) (xy 222.25 91.44)
-		)
-		(stroke
-			(width 0)
-			(type default)
-		)
-	)
-	(wire
-		(pts
 			(xy 78.74 45.72) (xy 97.79 45.72)
 		)
@@
 	(wire
 		(pts
-			(xy 44.45 107.95) (xy 44.45 110.49)
+			(xy 200.66 66.04) (xy 200.66 46.99)
 		)
 		(stroke
@@
 	(wire
 		(pts
-			(xy 204.47 44.45) (xy 198.12 44.45)
+			(xy 44.45 107.95) (xy 44.45 110.49)
 		)
 		(stroke
@@
 	(wire
 		(pts
-			(xy 180.34 41.91) (xy 180.34 54.61)
+			(xy 220.98 39.37) (xy 220.98 88.9)
 		)
 		(stroke
@@
 	(wire
 		(pts
+			(xy 198.12 44.45) (xy 198.12 66.04)
+		)
+		(stroke
+			(width 0)
+			(type default)
+		)
+	)
+	(wire
+		(pts
 			(xy 157.48 50.8) (xy 157.48 101.6)
 		)
@@
 	(wire
 		(pts
+			(xy 222.25 91.44) (xy 222.25 44.45)
+		)
+		(stroke
+			(width 0)
+			(type default)
+		)
+	)
+	(wire
+		(pts
 			(xy 76.2 59.69) (xy 76.2 49.53)
 		)
@@
 	(wire
 		(pts
-			(xy 198.12 44.45) (xy 198.12 66.04)
-		)
-		(stroke
-			(width 0)
-			(type default)
-		)
-	)
-	(wire
-		(pts
 			(xy 165.1 134.62) (xy 165.1 147.32)
 		)
@@
 	(wire
 		(pts
+			(xy 200.66 46.99) (xy 203.2 46.99)
+		)
+		(stroke
+			(width 0)
+			(type default)
+		)
+	)
+	(wire
+		(pts
+			(xy 203.2 39.37) (xy 203.2 41.91)
+		)
+		(stroke
+			(width 0)
+			(type default)
+		)
+	)
+	(wire
+		(pts
 			(xy 101.6 77.47) (xy 105.41 77.47)
 		)
@@
 	(wire
 		(pts
-			(xy 217.17 46.99) (xy 220.98 46.99)
+			(xy 147.32 128.27) (xy 146.05 128.27)
 		)
 		(stroke
@@
 	(wire
 		(pts
-			(xy 147.32 128.27) (xy 146.05 128.27)
+			(xy 27.94 85.09) (xy 27.94 90.17)
 		)
 		(stroke
@@
 	(wire
 		(pts
-			(xy 27.94 85.09) (xy 27.94 90.17)
+			(xy 86.36 123.19) (xy 76.2 123.19)
 		)
 		(stroke
@@
 	(wire
 		(pts
-			(xy 86.36 123.19) (xy 76.2 123.19)
+			(xy 59.69 133.35) (xy 59.69 135.89)
 		)
 		(stroke
@@
 	(wire
 		(pts
-			(xy 204.47 46.99) (xy 200.66 46.99)
+			(xy 49.53 69.85) (xy 49.53 68.58)
 		)
 		(stroke
@@
 	(wire
 		(pts
-			(xy 59.69 133.35) (xy 59.69 135.89)
+			(xy 55.88 77.47) (xy 60.96 77.47)
 		)
 		(stroke
@@
 	(wire
 		(pts
-			(xy 49.53 69.85) (xy 49.53 68.58)
+			(xy 88.9 35.56) (xy 88.9 41.91)
 		)
 		(stroke
@@
 	(wire
 		(pts
-			(xy 55.88 77.47) (xy 60.96 77.47)
+			(xy 222.25 44.45) (xy 215.9 44.45)
 		)
 		(stroke
@@
 	(wire
 		(pts
-			(xy 88.9 35.56) (xy 88.9 41.91)
+			(xy 198.12 44.45) (xy 203.2 44.45)
 		)
 		(stroke
@@
 	(wire
 		(pts
-			(xy 220.98 46.99) (xy 220.98 88.9)
-		)
-		(stroke
-			(width 0)
-			(type default)
-		)
-	)
-	(wire
-		(pts
 			(xy 53.34 124.46) (xy 59.69 124.46)
 		)
@@
 	(symbol
 		(lib_id "Connector_Generic:Conn_02x03_Counter_Clockwise")
-		(at 209.55 44.45 0)
+		(at 210.82 44.45 180)
 		(unit 1)
 		(exclude_from_sim no)
@@
 		(fields_autoplaced yes)
 		(property "Reference" "J2"
-			(at 210.82 35.56 0)
+			(at 209.55 38.1 0)
 			(effects
 				(font
@@
 		)
 		(property "Value" "Conn_02x03_Counter_Clockwise"
-			(at 210.82 38.1 0)
+			(at 209.55 50.8 0)
 			(effects
 				(font
@@
 			)
 		)
-		(property "Footprint" "Connector_PinHeader_2.54mm:PinHeader_2x03_P2.54mm_Vertical"
-			(at 209.55 44.45 0)
+		(property "Footprint" "Connector_PinHeader_1.27mm:PinHeader_2x03_P1.27mm_Vertical"
+			(at 210.82 44.45 0)
 			(effects
 				(font
@@
 		)
 		(property "Datasheet" "~"
-			(at 209.55 44.45 0)
+			(at 210.82 44.45 0)
 			(effects
 				(font
@@
 		)
 		(property "Description" "Generic connector, double row, 02x03, counter clockwise pin numbering scheme (similar to DIP package numbering), script generated (kicad-library-utils/schlib/autogen/connector/)"
-			(at 209.55 44.45 0)
+			(at 210.82 44.45 0)
 			(effects
 				(font
@@
 			)
 		)
-		(property "Footprint" "Crystal:Crystal_SMD_3225-4Pin_3.2x2.5mm_HandSoldering"
+		(property "Footprint" "Crystal:Crystal_SMD_3225-4Pin_3.2x2.5mm"
 			(at 85.09 35.56 0)
 			(effects
@@
 			)
 		)
-		(property "Footprint" "Library:QFN50P500X500X60-33N-D"
+		(property "Footprint" "Package_DFN_QFN:UQFN-32_5x5mm_P0.5mm"
 			(at 212.09 168.58 0)
 			(effects

Commit message: Update
Parts:
- J3, J4: footprint Connector_PinHeader_2.54mm:PinHeader_1x10_P2.54mm_Vertical -> Connector_PinHeader_2.54mm:PinHeader_1x11_P2.54mm_Vertical; symbol Connector_Generic:Conn_01x10 -> Connector_Generic:Conn_01x11
Connections:
- net 12V: now also J4.11 (Pin_11); no longer J4.10 (Pin_10)
- net 3V3: now also J4.2 (Pin_2); no longer J4.1 (Pin_1)
- net GND: now also J4.10 (Pin_10); no longer IC1.33 (EP), J4.9 (Pin_9)
- net at IC1.13 (PB0): now also J4.3 (Pin_3); no longer J4.2 (Pin_2)
- net at IC1.12 (PA7): now also J4.4 (Pin_4); no longer J4.3 (Pin_3)
- net at IC1.11 (PA6): now also J4.5 (Pin_5); no longer J4.4 (Pin_4)
- net at IC1.10 (PA5): now also J4.6 (Pin_6); no longer J4.5 (Pin_5)
- net at IC1.9 (PA4): now also J4.7 (Pin_7); no longer J4.6 (Pin_6)
- net at IC1.4 (PG10-NRST), R6.2: now also J4.8 (Pin_8); no longer J4.7 (Pin_7)
- net at IC1.2 (RCC_OSC_IN), IC2.32 (XCLK): now also J4.9 (Pin_9); no longer J4.8 (Pin_8)
- net at IC1.26 (DEBUG_TX), J2.5 (Pin_5): now also J3.11 (Pin_11)
- net at IC1.25 (DEBUG_RX), J2.6 (Pin_6): now also J4.1 (Pin_1)

Commit message: Fix Error (First JLCPCB board was fail)
Parts:
- C1, C2, C3, C4, C5, C6, C7, C8, C9: JLCPCB (none) -> C2189775
- C10: JLCPCB (none) -> C668335
- C11, C12: JLCPCB (none) -> C109040
- C13, C14: JLCPCB (none) -> C76946
- C15: JLCPCB (none) -> C2188111
- C16: JLCPCB (none) -> C2169603
- C17: JLCPCB (none) -> C7442652
- D1: JLCPCB (none) -> C113257
- D2: JLCPCB (none) -> C19077552
- D3: JLCPCB (none) -> C6067128
- IC1: JLCPCB (none) -> C3225629
- IC2: JLCPCB (none) -> C513000
- L1, L2: JLCPCB (none) -> C223324
- R1: JLCPCB (none) -> C1884631
- R10: JLCPCB (none) -> C25478
- R11, R9: JLCPCB (none) -> C2077491
- R2: JLCPCB (none) -> C482096
- R3: JLCPCB (none) -> C2654005
- R4, R5, R6, R7: JLCPCB (none) -> C2654001
- R8: JLCPCB (none) -> C481961
- SW1: JLCPCB (none) -> C115351
- Y1: JLCPCB (none) -> C164044
Connections:
- net 3V3: now also C3.1, IC2.40 (VDDA); no longer IC2.31 (VSSD)
- net GND: now also C13.2, C14.2, IC2.31 (VSSD)
- net at C17.1, C6.1, IC2.9 (VFILT): now also IC2.16 (VIN)
- net at C10.1, IC2.10 (V20V): no longer IC2.16 (VIN)
Other:
- moved on the sheet: C13, C14, C4, R3

Commit message: After review
Parts:
- removed R3: 10k, Resistor_SMD:R_0402_1005Metric, symbol Device:R
- added C18: 0.1 uF 50 VDC 5% 0402 X7S, Capacitor_SMD:C_0402_1005Metric, symbol Device:C
- added FID1, FID2, FID3: Fiducial, Fiducial:Fiducial_1mm_Mask2mm, symbol Mechanical:Fiducial
- C11: value 10 uF 16 VDC 10% 0805 X7S -> 22 uF 25 VDC 0805 X5R; JLCPCB C109040 -> C398931; Manufacturer_Part_Number GRM21BC71E106KE11L -> GRT21BR61E226ME13L
Connections:
- net GND: now also J2.3 (Pin_3), C18.2
- net at R4.2: now also IC1.8 (KNX_RX); no longer IC1.7 (KNX_TX)
- net at IC1.4 (PG10-NRST), J4.8 (Pin_8), R6.2: now also C18.1
- net at R5.2: now also IC1.7 (KNX_TX); no longer IC1.8 (KNX_RX)
