File: hardware/KnxBoard.sch (KiCad schematic (older format))
At the start: 40 parts, among them J1 Conn_01x10, J2 Conn_01x12, J3 Conn_01x12, J4 Conn_01x02_Male, U1 NCN5130, U2 STM32L432KCUx, X1 FA-238

Commit message: Update BOM
Parts:
- C4: MPN UUR1V101MCL6GS -> EMZA350ADA101MF80S
- C8, C9: MPN CL10C100JB8NNND -> CL10C100DB81PNC
- R2, R3: MPN CRCW06031R00JNEC -> SFR03EZPJ1R0
- R20: Price 0.085 -> 0.078
- R4: MPN MCT06030C5602FP500 -> RT0603DRE0756KL; Price 0.08 -> 0.078
- R5: MPN MCT06030C4993FP500 -> RT0603FRE07499KL; Price 0.102 -> 0.059
- X1: MPN FA-238 16.0000MD30X-W3 -> FA-238 16.0000MB-K3; Price 0.445 -> 0.464
Changed lines of the file:
@@
 F 1 "100uF 35V" H 1968 4105 50  0001 L CNN
 F 2 "Capacitor_SMD:CP_Elec_6.3x7.7" H 1888 4000 50  0001 C CNN
-F 3 "https://www.mouser.fr/ProductDetail/Nichicon/UUR1V101MCL6GS?qs=huzeVNXgovWypttWSImRTA%3D%3D" H 1850 4150 50  0001 C CNN
+F 3 "https://www.mouser.fr/ProductDetail/United-Chemi-Con-UCC/EMZA350ADA101MF80S?qs=sGAEpiMZZMv0fKVy8cA0DeAj7ZPp8rk3i6NetwAXjI0%3D" H 1850 4150 50  0001 C CNN
 F 4 "0.353" H 1850 4150 50  0001 C CNN "Price"
-F 5 "UUR1V101MCL6GS " H 1850 4150 50  0001 C CNN "MPN"
+F 5 "EMZA350ADA101MF80S " H 1850 4150 50  0001 C CNN "MPN"
 	1    1850 4150
 	1    0    0    -1
@@
 F 1 "56K 1/16w" V 2784 4750 50  0001 C CNN
 F 2 "Resistor_SMD:R_0603_1608Metric" V 2830 4750 50  0001 C CNN
-F 3 "https://www.mouser.fr/ProductDetail/Vishay-Beyschlag/MCT06030C5602FP500?qs=sGAEpiMZZMvdGkrng054txcf3av6vnC8XzTnB3mS7jw%3D" H 2900 4750 50  0001 C CNN
-F 4 "0.08" H 2900 4750 50  0001 C CNN "Price"
-F 5 "MCT06030C5602FP500 " H 2900 4750 50  0001 C CNN "MPN"
+F 3 "https://www.mouser.fr/ProductDetail/YAGEO/RT0603DRE0756KL?qs=4CyHz7GXqSjwr563n0hfGQ%3D%3D" H 2900 4750 50  0001 C CNN
+F 4 "0.078" H 2900 4750 50  0001 C CNN "Price"
+F 5 "RT0603DRE0756KL " H 2900 4750 50  0001 C CNN "MPN"
 	1    2900 4750
 	-1   0    0    1
@@
 F 1 "499K 1/16w" V 2784 5250 50  0001 C CNN
 F 2 "Resistor_SMD:R_0603_1608Metric" V 2830 5250 50  0001 C CNN
-F 3 "https://www.mouser.fr/ProductDetail/Vishay-Beyschlag/MCT06030C4993FP500?qs=8lczJKL2ryeXiIiBeB6JCA%3D%3D" H 2900 5250 50  0001 C CNN
-F 4 "0.102" H 2900 5250 50  0001 C CNN "Price"
-F 5 "MCT06030C4993FP500 " H 2900 5250 50  0001 C CNN "MPN"
+F 3 "https://www.mouser.fr/ProductDetail/YAGEO/RT0603FRE07499KL?qs=%2Ff7pOCXLR5dHyFF6GLQcKQ%3D%3D" H 2900 5250 50  0001 C CNN
+F 4 "0.059" H 2900 5250 50  0001 C CNN "Price"
+F 5 "RT0603FRE07499KL " H 2900 5250 50  0001 C CNN "MPN"
 	1    2900 5250
 	-1   0    0    1
@@
 F 1 "1R 1/16W" V 3234 4850 50  0001 C CNN
 F 2 "Resistor_SMD:R_0603_1608Metric" V 3280 4850 50  0001 C CNN
-F 3 "https://www.mouser.fr/ProductDetail/Vishay-Dale/CRCW06031R00JNEC?qs=sGAEpiMZZMvdGkrng054t8tsKUCh5%2FbY4AhBMsyzAQQ%3D" H 3350 4850 50  0001 C CNN
+F 3 "https://www.mouser.fr/ProductDetail/ROHM-Semiconductor/SFR03EZPJ1R0?qs=Mv7BduZupUhg%2FozxqD6EfA%3D%3D" H 3350 4850 50  0001 C CNN
 F 4 "0.008" H 3350 4850 50  0001 C CNN "Price"
-F 5 "CRCW06031R00JNEC " H 3350 4850 50  0001 C CNN "MPN"
+F 5 "SFR03EZPJ1R0" H 3350 4850 50  0001 C CNN "MPN"
 	1    3350 4850
 	-1   0    0    1
@@
 F 1 "1R 1/16W" V 3834 4850 50  0001 C CNN
 F 2 "Resistor_SMD:R_0603_1608Metric" V 3880 4850 50  0001 C CNN
-F 3 "https://www.mouser.fr/ProductDetail/Vishay-Dale/CRCW06031R00JNEC?qs=sGAEpiMZZMvdGkrng054t8tsKUCh5%2FbY4AhBMsyzAQQ%3D" H 3950 4850 50  0001 C CNN
+F 3 "https://www.mouser.fr/ProductDetail/ROHM-Semiconductor/SFR03EZPJ1R0?qs=Mv7BduZupUhg%2FozxqD6EfA%3D%3D" H 3950 4850 50  0001 C CNN
 F 4 "0.008" H 3950 4850 50  0001 C CNN "Price"
-F 5 "CRCW06031R00JNEC " H 3950 4850 50  0001 C CNN "MPN"
+F 5 "SFR03EZPJ1R0" H 3950 4850 50  0001 C CNN "MPN"
 	1    3950 4850
 	-1   0    0    1
@@
 F 1 "10pF 6.3V" V 3389 1450 50  0001 C CNN
 F 2 "Capacitor_SMD:C_0603_1608Metric" H 3588 1300 50  0001 C CNN
-F 3 "https://www.mouser.fr/ProductDetail/Samsung-Electro-Mechanics/CL10C100JB8NNND?qs=sGAEpiMZZMvsSlwiRhF8qlxW52pIu5FNW3qxrQ2K0NU%3D" H 3550 1450 50  0001 C CNN
+F 3 "https://www.mouser.fr/ProductDetail/Samsung-Electro-Mechanics/CL10C100DB81PNC?qs=sGAEpiMZZMvsSlwiRhF8qtsGU%2FCnaNeQ%252BDo2JdVgb2ygiVq9388VOw%3D%3D" H 3550 1450 50  0001 C CNN
 F 4 "0.032" H 3550 1450 50  0001 C CNN "Price"
-F 5 "CL10C100JB8NNND " H 3550 1450 50  0001 C CNN "MPN"
+F 5 "CL10C100DB81PNC" H 3550 1450 50  0001 C CNN "MPN"
 	1    3550 1450
 	1    0    0    -1
@@
 F 1 "10pF 6.3V" V 3689 1450 50  0001 C CNN
 F 2 "Capacitor_SMD:C_0603_1608Metric" H 3888 1300 50  0001 C CNN
-F 3 "https://www.mouser.fr/ProductDetail/Samsung-Electro-Mechanics/CL10C100JB8NNND?qs=sGAEpiMZZMvsSlwiRhF8qlxW52pIu5FNW3qxrQ2K0NU%3D" H 3850 1450 50  0001 C CNN
+F 3 "https://www.mouser.fr/ProductDetail/Samsung-Electro-Mechanics/CL10C100DB81PNC?qs=sGAEpiMZZMvsSlwiRhF8qtsGU%2FCnaNeQ%252BDo2JdVgb2ygiVq9388VOw%3D%3D" H 3850 1450 50  0001 C CNN
 F 4 "0.032" H 3850 1450 50  0001 C CNN "Price"
-F 5 "CL10C100JB8NNND " H 3850 1450 50  0001 C CNN "MPN"
+F 5 "CL10C100DB81PNC" H 3850 1450 50  0001 C CNN "MPN"
 	1    3850 1450
 	1    0    0    -1
@@
 F 1 "FA-238" H 3894 1855 50  0000 L CNN
 F 2 "Crystal:Crystal_SMD_SeikoEpson_FA238-4Pin_3.2x2.5mm" H 3700 1900 50  0001 C CNN
-F 3 "https://www.mouser.fr/ProductDetail/Epson-Timing/FA-238-160000MD30X-W3?qs=f9yNj16SXrIs1foPi9xf%2Fw%3D%3D" H 3700 1900 50  0001 C CNN
-F 4 "0.445" H 3700 1900 50  0001 C CNN "Price"
-F 5 "FA-238 16.0000MD30X-W3 " H 3700 1900 50  0001 C CNN "MPN"
+F 3 "https://www.mouser.fr/ProductDetail/Epson-Timing/FA-238-160000MB-K3?qs=CANAagUtPAoF3w0fRAI0xg%3D%3D" H 3700 1900 50  0001 C CNN
+F 4 "0.464" H 3700 1900 50  0001 C CNN "Price"
+F 5 "FA-238 16.0000MB-K3" H 3700 1900 50  0001 C CNN "MPN"
 	1    3700 1900
 	1    0    0    -1
@@
 F 2 "Resistor_SMD:R_0603_1608Metric" V 7680 3300 50  0001 C CNN
 F 3 "https://www.mouser.fr/ProductDetail/Vishay-Beyschlag/MCT06030C1002FP500?qs=sGAEpiMZZMvdGkrng054t%252B7N8nKX0VXe%2FafJHKs0Nqw%3D" H 7750 3300 50  0001 C CNN
-F 4 "0.085" H 7750 3300 50  0001 C CNN "Price"
+F 4 "0.078" H 7750 3300 50  0001 C CNN "Price"
 F 5 "MCT06030C1002FP500 " H 7750 3300 50  0001 C CNN "MPN"
 	1    7750 3300
