File: hardware/knxncn.kicad_sch (KiCad schematic)
At the start: 28 parts, among them IC1 NCN5130, J4 Conn_01x02, X1 FA-238

Commit message: Seed SeeedStudio N°1
Connections:
- net +3V3: no longer IC1.21 (XCLKC)
- net at JP1.2 (C): now also IC1.21 (XCLKC); no longer IC1.33 (XSEL)
- no-connect marks 2 -> 3
Other:
- moved on the sheet: JP1
Changed lines of the file:
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@@
   (junction (at 109.22 99.06) (diameter 0) (color 0 0 0 0)
   )
+  (no_connect (at 142.24 60.96))
   (no_connect (at 154.94 99.06))
   (no_connect (at 127 60.96))
@@
     (stroke (width 0) (type default) (color 0 0 0 0))
   )
+  (wire (pts (xy 167.64 101.6) (xy 167.64 104.14))
+    (stroke (width 0) (type default) (color 0 0 0 0))
+  )
   (wire (pts (xy 144.78 58.42) (xy 168.91 58.42))
     (stroke (width 0) (type default) (color 0 0 0 0))
@@
     (stroke (width 0) (type default) (color 0 0 0 0))
   )
+  (wire (pts (xy 154.94 101.6) (xy 167.64 101.6))
+    (stroke (width 0) (type default) (color 0 0 0 0))
+  )
   (wire (pts (xy 142.24 22.86) (xy 134.62 22.86))
     (stroke (width 0) (type default) (color 0 0 0 0))
   )
-  (wire (pts (xy 142.24 50.8) (xy 142.24 60.96))
-    (stroke (width 0) (type default) (color 0 0 0 0))
-  )
   (wire (pts (xy 127 130.81) (xy 127 128.27))
     (stroke (width 0) (type default) (color 0 0 0 0))
@@
   )
   (wire (pts (xy 110.49 78.74) (xy 114.3 78.74))
-    (stroke (width 0) (type default) (color 0 0 0 0))
-  )
-  (wire (pts (xy 152.4 50.8) (xy 142.24 50.8))
     (stroke (width 0) (type default) (color 0 0 0 0))
   )
@@
     (effects (font (size 1.27 1.27)) (justify left))
   )
-  (symbol (lib_id "Jumper:SolderJumper_3_Bridged12") (at 152.4 46.99 0) (unit 1)
-    (in_bom yes) (on_board yes)
-    (property "Reference" "JP1" (id 0) (at 152.4 44.45 0))
-    (property "Value" "Clock_8_16" (id 1) (at 152.4 43.18 0)
-      (effects (font (size 1.27 1.27)) hide)
-    )
-    (property "Footprint" "Jumper:SolderJumper-3_P1.3mm_Open_RoundedPad1.0x1.5mm" (id 2) (at 152.4 46.99 0)
-      (effects (font (size 1.27 1.27)) hide)
-    )
-    (property "Datasheet" "~" (id 3) (at 152.4 46.99 0)
+  (symbol (lib_id "Jumper:SolderJumper_3_Bridged12") (at 167.64 107.95 180) (unit 1)
+    (in_bom yes) (on_board yes)
+    (property "Reference" "JP1" (id 0) (at 167.64 110.49 0))
+    (property "Value" "Clock_8_16" (id 1) (at 167.64 111.76 0)
+      (effects (font (size 1.27 1.27)) hide)
+    )
+    (property "Footprint" "Jumper:SolderJumper-3_P1.3mm_Open_RoundedPad1.0x1.5mm" (id 2) (at 167.64 107.95 0)
+      (effects (font (size 1.27 1.27)) hide)
+    )
+    (property "Datasheet" "~" (id 3) (at 167.64 107.95 0)
       (effects (font (size 1.27 1.27)) hide)
     )
@@
     )
     (property "Datasheet" "" (id 3) (at 132.08 43.18 0)
-      (effects (font (size 1.27 1.27)) hide)
-    )
-    (pin "1")
-  )
-  (symbol (lib_id "power:+3V3") (at 154.94 101.6 270) (unit 1)
-    (in_bom yes) (on_board yes) (fields_autoplaced)
-    (property "Reference" "#PWR0129" (id 0) (at 151.13 101.6 0)
-      (effects (font (size 1.27 1.27)) hide)
-    )
-    (property "Value" "+3V3" (id 1) (at 158.75 101.5999 90)
-      (effects (font (size 1.27 1.27)) (justify left))
-    )
-    (property "Footprint" "" (id 2) (at 154.94 101.6 0)
-      (effects (font (size 1.27 1.27)) hide)
-    )
-    (property "Datasheet" "" (id 3) (at 154.94 101.6 0)
       (effects (font (size 1.27 1.27)) hide)
     )
@@
     (pin "2")
   )
-  (symbol (lib_id "power:+3V3") (at 157.48 46.99 270) (unit 1)
+  (symbol (lib_id "power:+3V3") (at 162.56 107.95 90) (unit 1)
     (in_bom yes) (on_board yes) (fields_autoplaced)
-    (property "Reference" "#PWR0141" (id 0) (at 153.67 46.99 0)
-      (effects (font (size 1.27 1.27)) hide)
-    )
-    (property "Value" "+3V3" (id 1) (at 161.29 46.9899 90)
-      (effects (font (size 1.27 1.27)) (justify left))
-    )
-    (property "Footprint" "" (id 2) (at 157.48 46.99 0)
-      (effects (font (size 1.27 1.27)) hide)
-    )
-    (property "Datasheet" "" (id 3) (at 157.48 46.99 0)
+    (property "Reference" "#PWR0141" (id 0) (at 166.37 107.95 0)
+      (effects (font (size 1.27 1.27)) hide)
+    )
+    (property "Value" "+3V3" (id 1) (at 158.75 107.9501 90)
+      (effects (font (size 1.27 1.27)) (justify left))
+    )
+    (property "Footprint" "" (id 2) (at 162.56 107.95 0)
+      (effects (font (size 1.27 1.27)) hide)
+    )
+    (property "Datasheet" "" (id 3) (at 162.56 107.95 0)
       (effects (font (size 1.27 1.27)) hide)
     )
@@
     (pin "2")
   )
-  (symbol (lib_id "power:GNDREF") (at 147.32 46.99 270) (unit 1)
-    (in_bom yes) (on_board yes)
-    (property "Reference" "#PWR0139" (id 0) (at 140.97 46.99 0)
-      (effects (font (size 1.27 1.27)) hide)
-    )
-    (property "Value" "GNDREF" (id 1) (at 144.78 49.53 90))
-    (property "Footprint" "" (id 2) (at 147.32 46.99 0)
-      (effects (font (size 1.27 1.27)) hide)
-    )
-    (property "Datasheet" "" (id 3) (at 147.32 46.99 0)
-      (effects (font (size 1.27 1.27)) hide)
-    )
+  (symbol (lib_id "power:GNDREF") (at 172.72 107.95 90) (unit 1)
+    (in_bom yes) (on_board yes)
+    (property "Reference" "#PWR0139" (id 0) (at 179.07 107.95 0)
+      (effects (font (size 1.27 1.27)) hide)
+    )
+    (property "Value" "GNDREF" (id 1) (at 175.26 105.41 90))
+    (property "Footprint" "" (id 2) (at 172.72 107.95 0)
+      (effects (font (size 1.27 1.27)) hide)
+    )
+    (property "Datasheet" "" (id 3) (at 172.72 107.95 0)
+      (effects (font (size 1.27 1.27)) hide)
+    )

Commit message: State: Led Blink on both Nucleo and KnxBoardV3
Parts:
- C10: value 1uF 50V ESR < 2ohm -> 1uF 35V ESR < 2ohm
- C11: value 10uF 6.3V ESR < 0.1ohm -> 10uF 16V ESR < 0.1ohm
Changed lines of the file:
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@@
       (effects (font (size 1.27 1.27)) (justify left))
     )
-    (property "Value" "10uF 6.3V ESR < 0.1ohm" (id 1) (at 110.871 140.843 0)
+    (property "Value" "10uF 16V ESR < 0.1ohm" (id 1) (at 110.871 140.843 0)
       (effects (font (size 1.27 1.27)) (justify left) hide)
     )
@@
       (effects (font (size 1.27 1.27)) (justify left))
     )
-    (property "Value" "1uF 50V ESR < 2ohm" (id 1) (at 100.711 109.093 0)
+    (property "Value" "1uF 35V ESR < 2ohm" (id 1) (at 100.711 109.093 0)
       (effects (font (size 1.27 1.27)) (justify left) hide)
     )
